File: CTR-0-main/CTR-0.kicad_pcb (KiCad board)
At the start: 2 copper layers, 21 x 51 mm, 38 parts, among them J1 USB_C_Receptacle_USB2.0_14P, J2 Conn_01x20, J3 Conn_01x20, J4 Conn_01x03, SW1 SW_Push, SW2 SW_Push, U1 RP2040, U2 NCP1117-3.3_SOT223, U3 W25Q128JVS, U4 TVS1400DRV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

Commit message: fix
footprints now obey drc, component graphics now obey drc
Routing:
- net GND: track 38.3 -> 0.20 mm, vias 8 -> 9
