File: CTR-0-main/CTR-0.kicad_pcb (KiCad board)
At the start: 2 copper layers, 21 x 51 mm, 38 parts, among them J1 USB_C_Receptacle_USB2.0_14P, J2 Conn_01x20, J3 Conn_01x20, J4 Conn_01x03, SW1 SW_Push, SW2 SW_Push, U1 RP2040, U2 NCP1117-3.3_SOT223, U3 W25Q128JVS, U4 TVS1400DRV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

Commit message: fixed footprints for bom
out of stock parts replaced
Parts:
- J1: footprint Connector_USB:USB_C_Receptacle_HRO_TYPE-C-31-M-12 -> Connector_USB:USB_C_Receptacle_GCT_USB4105-xx-A_16P_TopMnt_Horizontal
- moved J1 0.25 mm to (190.5, 72.7)
Routing:
- net +5V: track 30.5 -> 40.8 mm, vias 1 -> 0
