File: CTR-0-main/CTR-0.kicad_sch (KiCad schematic)
At the start: 38 parts, among them J1 USB_C_Receptacle_USB2.0_14P, J2 Conn_01x20, J3 Conn_01x20, J4 Conn_01x03, SW1 SW_Push, SW2 SW_Push, U1 RP2040, U2 NCP1117-3.3_SOT223, U3 W25Q128JVS, U4 TVS1400DRV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

Commit message: fixed footprints for bom
out of stock parts replaced
Parts:
- J1: footprint Connector_USB:USB_C_Receptacle_HRO_TYPE-C-31-M-12 -> Connector_USB:USB_C_Receptacle_GCT_USB4105-xx-A_16P_TopMnt_Horizontal
Changed lines of the file:
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@@
 			)
 		)
-		(property "Footprint" "Connector_USB:USB_C_Receptacle_HRO_TYPE-C-31-M-12"
+		(property "Footprint" "Connector_USB:USB_C_Receptacle_GCT_USB4105-xx-A_16P_TopMnt_Horizontal"
 			(at 49.53 49.53 0)
 			(hide yes)

Commit message: edit
updated footprints
Parts:
- U3: value W25Q128JVS -> MX25L12872FM2I-10G
- renumbered Y1 to YABM8-12.000MHZ-B2-T
Changed lines of the file:
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@@
 		(in_pos_files yes)
 		(dnp no)
-		(fields_autoplaced yes)
 		(property "Reference" "U3"
-			(at 119.38 57.1499 0)
+			(at 100.33 47.244 0)
 			(show_name no)
 			(do_not_autoplace no)
@@
 			)
 		)
-		(property "Value" "W25Q128JVS"
-			(at 119.38 59.6899 0)
+		(property "Value" "MX25L12872FM2I-10G"
+			(at 83.82 69.85 0)
 			(show_name no)
 			(do_not_autoplace no)
@@
 		(in_pos_files yes)
 		(dnp no)
-		(property "Reference" "Y1"
+		(property "Reference" "YABM8-12.000MHZ-B2-T"
 			(at 109.22 83.82 90)
 			(show_name no)
@@
 			(project "CTR-0"
 				(path "/68f715fb-4d48-413c-bc7b-70d6d6731680"
-					(reference "Y1")
-					(unit 1)
-				)
+					(reference "YABM8-12.000MHZ-B2-T")
+					(unit 1)
+				)
